File: handheld.kicad_pcb (KiCad board)
At the start: 2 copper layers, 170.4 x 140.6 mm, 19 parts, among them J1 Conn_01x15_Pin, J2 Conn_01x15_Pin, J3 Conn_02x13_Odd_Even, J6 Micro_SD_Card, SW1 SW_Push, SW10 SW_Push, SW11 SW_Push, SW12 SW_Push, SW2 SW_Push, SW3 SW_Push, SW4 SW_Push, SW5 SW_Push, SW6 SW_Push, SW7 SW_Push, SW8 SW_Push, SW9 SW_Push, U1 MCP23017x-x-SP

Commit message: updated sd card module
https://www.aliexpress.com/item/1005005302035188.html?spm=a2g0o.detail.pcDetailTopMoreOtherSeller.1.1d2a3a904oolQu&gps-id=pcDetailTopMoreOtherSeller&scm=1007.40050.354490.0&scm_id=1007.40050.354490.0&scm-url=1007.40050.354490.0&pvid=4e822c0b-3cde-49e3-9426-4f76b8918aef&_t=gps-id%3ApcDetailTopMoreOtherSeller%2Cscm-url%3A1007.40050.354490.0%2Cpvid%3A4e822c0b-3cde-49e3-9426-4f76b8918aef%2Ctpp_buckets%3A668%232846%238111%231996&pdp_ext_f=%7B%22order%22%3A%2210394%22%2C%22spu_best_type%22%3A%22price%22%2C%22eval%22%3A%221%22%2C%22sceneId%22%3A%2230050%22%2C%22fromPage%22%3A%22recommend%22%7D&pdp_npi=6%40dis%21GBP%210.58%210.55%21%21%210.76%210.72%21%400b0fe40d17872241439645102e0dfb%2112000032551641256%21rec%21UK%217739848304%21X%211%210%21n_tag%3A-29919%3Bd%3A1c53e4a4%3Bm03_new_user%3A-29895%3BpisId%3A5000000215431853&utparam-url=scene%3ApcDetailTopMoreOtherSeller%7Cquery_from%3A%7Cx_object_id%3A1005005302035188%7C_p_origin_prod%3A fyi
Parts:
- removed J6: Micro_SD_Card, Connector_Card:microSD_HC_Wuerth_693072010801
- removed R1, R2: 10K, Resistor_SMD:R_0805_2012Metric
- added J4: SD MODULE, Connector_PinHeader_2.54mm:PinHeader_1x06_P2.54mm_Vertical, F.Cu at (149.7, 143.8)
- moved SW4 92.7 mm to (42.1, 140.2)
- moved SW10 92.7 mm to (82.0, 117.0)
- moved SW5 92.7 mm to (102.7, 120.2)
- moved SW6 92.7 mm to (92.3, 130.0)
- moved SW8 92.7 mm to (102.5, 140.0)
- moved J1 92.7 mm to (167.5, 65.7)
- moved J2 92.7 mm to (139.6, 65.7)
- moved J3 92.7 mm to (40.4, 31.5)
- moved SW1 92.7 mm to (42.1, 120.1)
- moved SW11 92.7 mm to (27.8, 97.9)
- moved SW12 92.7 mm to (109.2, 97.3)
- moved SW2 92.7 mm to (32.1, 130.0)
- moved SW3 92.7 mm to (52.1, 130.0)
- moved SW7 92.7 mm to (113.8, 130.0)
- moved SW9 92.7 mm to (63.1, 117.1)
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Routing:
- net GND: track 1022.3 -> 946.3 mm
- net Net-(J6-DAT1): track 16.1 -> 0.00 mm
- net Net-(J6-DAT2): track 15.4 -> 0.00 mm
- net +3V3: track 602.9 -> 591.2 mm
- net /GPIO 19: track 210.1 -> 217.5 mm
- net /GPIO 23: track 189.8 -> 196.9 mm
- net /GPIO 18: track 200.4 -> 207.1 mm
- net /GPIO 14: track 177.4 -> 183.8 mm
Other:
- board text added: "3V3"
- board text added: "CLK"
- board text added: "CS"
- board text added: "GND"
- board text added: "MISO"
- board text added: "MOSI"

Commit message: final pcb
Routing:
- net GND: track 946.3 -> 925.0 mm
- net +5V: track 153.3 -> 152.4 mm
